File: flight-coms-board-flatsat.kicad_sch (KiCad schematic)
At the start: 50 parts, among them J2 Conn_02x05_Odd_Even, J3 Conn_02x10_Odd_Even, J4 Conn_02x10_Odd_Even, J5 CONSMA001-SMD-G, U1 CC1200, U2 TPS79330-EP, Y2 40MHz

Commit message: Add RP2350 and CC1200 SPI connections to schematic
Parts:
- removed A1: RaspberryPi_Pico, Module:RaspberryPi_Pico_Common_Unspecified, symbol MCU_Module:RaspberryPi_Pico
- added C10, C24, C30: 4.7u, symbol Device:C
- added C31, C35, C36, C37, C38, C39, C40, C41, C42, C43, C44, C47, C48, C49, C50: 100n, symbol Device:C
- added C45, C46: 15p, symbol Device:C
- added J1: JST Debug Connector, symbol Connector:Conn_01x05_Pin
- added L9: 3.3u, symbol Device:L
- added P1: USB_C_Plug_USB2.0, symbol Connector:USB_C_Plug_USB2.0
- added R1: 33, symbol Device:R
- added R3: 0, symbol Device:R
- added R6: 1k, symbol Device:R
- added R7, R8: 27, symbol Device:R
- added SW1: SW_Push, symbol Switch:SW_Push
- added U3: RP2350B-QFN80, symbol rp2350b-qfn80:RP2350B-QFN80
- added U4: W25Q128JVS, Package_SO:SOIC-8_5.3x5.3mm_P1.27mm, symbol Memory_Flash:W25Q128JVS
- added Y1: Abracon ABM8-272-T3, symbol Device:Crystal_GND24
Connections:
- net CSN: now also U3.2 (GPIO5)
- net GND: now also C10.2, C24.1, C30.1, C31.1, C35.1, C36.1, C37.1, C38.1, C39.1, C40.1, C41.2, C42.2, C43.2, C44.1, C45.1, C46.1, C47.1, C48.1, C49.1, C50.1, J1.5 (Pin_5), SW1.1, U3.62 (VREG_PGND), U3.81 (GND), Y1.2 (G), Y1.4 (G)
- net GPIO0: now also U3.78 (GPIO1)
- net GPIO2: now also U3.79 (GPIO2)
- net GPIO3: now also U3.80 (GPIO3)
- net MISO: now also U3.1 (GPIO4)
- net MOSI: now also U3.4 (GPIO7)
- net RESET: now also U3.77 (GPIO0)
- net SCLK: now also U3.3 (GPIO6)
- net at C15.1, L3.1, U1.17 (PA): now also C22.1, L6.2, L7.1, U1.20 (LNA_N)
- new net: R7.2, U3.67 (USB_DP)
- new net: C10.1, R1.2, U3.61 (VREG_AVDD)
- new net: L9.1, U3.63 (VREG_LX)
- new net: R8.2, U3.66 (USB_DM)
- new net: P1.A1 (GND), P1.A12 (GND), P1.B1 (GND), P1.B12 (GND)
- new net: P1.A4 (VBUS), P1.A9 (VBUS), P1.B4 (VBUS), P1.B9 (VBUS)
- new net: J1.2 (Pin_2), J1.4 (Pin_4)
- new net +1V1: C24.2, C41.1, C42.1, C43.1, L9.2, U3.10 (DVDD), U3.32 (DVDD), U3.51 (DVDD), U3.65 (VREG_FB)
- new net +3V3: C30.2, C31.2, C35.2, C36.2, C37.2, C38.2, C39.2, C40.2, C44.2, C47.2, C48.2, C49.2, C50.2, R1.1, R3.2, U3.15 (IOVDD), U3.24 (IOVDD), U3.29 (IOVDD), U3.41 (IOVDD), U3.5 (IOVDD), U3.50 (IOVDD), U3.59 (ADC_AVDD), U3.60 (IOVDD), U3.64 (VREG_VIN), U3.68 (USB_OTP_VDD), U3.76 (IOVDD), U4.1 (~{CS}), U4.8 (VCC)
- new net QSPI_SCLK: U3.71 (QSPI_SCLK), U4.6 (CLK)
- new net QSPI_SD0: U3.72 (QSPI_SD0), U4.5 (DI/IO_{0})
- new net QSPI_SD1: U3.74 (QSPI_SD1), U4.2 (DO/IO_{1})
- new net QSPI_SD2: U3.73 (QSPI_SD2), U4.3 (~{WP}/IO_{2})
- new net QSPI_SD3: U3.70 (QSPI_SD3), U4.7 (~{HOLD}/~{RESET}/IO_{3})
- new net QSPI_SS: R3.1, R6.1, U3.75 (QSPI_SS)
- new net SWCLK: J1.1 (Pin_1), U3.33 (SWCLK)
- new net SWDIO: J1.3 (Pin_3), U3.34 (SWDIO)
- new net USB_BOOT: R6.2, SW1.2
- new net USB_DM: P1.A7 (D-), R8.1
- new net USB_DP: P1.A6 (D+), R7.1
- new net XIN: C45.2, U3.30 (XIN), Y1.1
- new net XOUT: C46.2, U3.31 (XOUT), Y1.3
- no-connect marks 56 -> 28
Other:
- note added: "12MHz Oscillator"
- note added: "BOOTSEL Button"
- note added: "Flash"
- moved on the sheet: C21, C22, L5, L6, L7, L8

Commit message: added external PA and RF switch
Parts:
- removed L5: 15nH, Inductor_SMD:L_0402_1005Metric_Pad0.77x0.64mm_HandSolder, symbol Device:L
- removed P1: USB_C_Plug_USB2.0, symbol Connector:USB_C_Plug_USB2.0
- added C51: 4.7u, symbol Device:C
- added C52, C56, C63, C65: 10000pF, Capacitor_SMD:C_0402_1005Metric, symbol Device:C
- added C53, C58, C70: 1000pF, Capacitor_SMD:C_0402_1005Metric, symbol Device:C
- added C54, C69: 3.3uF, Capacitor_SMD:C_1206_3216Metric, symbol Device:C
- added C55, C57, C62, C64, C66, C68: DNP, symbol Device:C
- added C59, C75: 56pF, Capacitor_SMD:C_0402_1005Metric, symbol Device:C
- added C60, C61: 330pF, Capacitor_SMD:C_0402_1005Metric, symbol Device:C
- added C67: 100pF, Capacitor_SMD:C_0402_1005Metric, symbol Device:C
- added C71: 47pF, Capacitor_SMD:C_0402_1005Metric, symbol Device:C
- added C72: 27pF, Capacitor_SMD:C_0402_1005Metric, symbol Device:C
- added C73: 22pF, Capacitor_SMD:C_0402_1005Metric, symbol Device:C
- added C74: 2pF, Capacitor_SMD:C_0402_1005Metric, symbol Device:C
- added IC1: QPA9510SB, QFN50P300X300X90-17N-D, symbol QPA9510SB:QPA9510SB
- added J6: USB_C_Receptacle_USB2.0_16P, symbol Connector:USB_C_Receptacle_USB2.0_16P
- added L11, L12: 0, Resistor_SMD:R_0402_1005Metric, symbol Device:L
- added L13: 12nH, Capacitor_SMD:C_0603_1608Metric, symbol Device:L
- added L14: 6.8nH, Capacitor_SMD:C_0603_1608Metric, symbol Device:L
- added L15: 1uH, Resistor_SMD:R_0603_1608Metric, symbol Device:L
- added L16: 2.4nH, Diode_SMD:D_0603_1608Metric, symbol Device:L
- added R10, R9: 5.1k, symbol Device:R
- added R11: 1M, symbol Device:R
- added R12: 180, symbol Device:R
- added R13, R14: 0, Resistor_SMD:R_0402_1005Metric, symbol Device:R
- added R15: 1k, symbol Device:R
- added R16: 5.6k, symbol Device:R
- added R17, R19: 10k, symbol Device:R
- added R18, R20: 33k, symbol Device:R
- added U5: SKY13330-397LF, QFN_330-397LF_SKY, symbol 2026-10-23_22-32-40:SKY13330-397LF
Connections:
- net 3V3: now also C52.1, C53.1, C54.1, C56.1, C58.1, C67.2, C69.1, C70.1, C71.1, IC1.14 (VCC), L11.1, L12.2, L15.2, U5.9 (VBATT)
- net GND: now also C23.1, J1.2 (Pin_2), J1.4 (Pin_4), C51.2, C52.2, C53.2, C54.2, C55.2, C56.2, C57.2, C58.2, C60.2, C61.2, C62.2, C63.2, C64.2, C65.1, C66.2, C67.1, C68.2, C69.2, C70.2, C71.2, C72.2, C73.2, C74.2, IC1.17 (GND), IC1.2 (GND1), IC1.4 (GND2), J6.A1 (GND), J6.A12 (GND), J6.B1 (GND), J6.B12 (GND), R10.1, R11.2, R12.2, R16.1, R18.1, R20.1, R9.2
- net GPIO0: no longer U3.78 (GPIO1)
- net GPIO2: now also R17.2; no longer U3.79 (GPIO2)
- net GPIO3: now also R15.2; no longer U3.80 (GPIO3)
- net USB_DM: now also J6.A7 (D-), J6.B7 (D-)
- net USB_DP: now also J6.A6 (D+), J6.B6 (D+)
- net at C22.1, L6.2, L7.1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: no longer C15.1, L3.1, U1.17 (PA)
- net at U1.18 (TRX_SW): no longer C23.1
- net RX: now reaches C21.1, L6.1
- net RX: now also U5.11 (RF2)
- net PA: now reaches C29.2, L4.2
- net PA: now also C59.1, R12.1; no longer J5.2
- new net: C65.2, IC1.15 (APC2), R13.2, R14.1
- new net: C15.1, L3.1, U1.17 (PA)
- new net: C73.1, C74.1, C75.1, L16.1
- new net: C62.1, C64.1, IC1.5 (VCC2_1), IC1.6 (VCC2_2), IC1.7 (NC_1), L14.2
- new net: C55.1, C57.1, C60.1, L12.1, L13.1
- new net: J6.B5 (CC2), R10.2
- new net: C68.1, C72.1, IC1.10 (RF_OUT_2), IC1.11 (RF_OUT_3), IC1.12 (RF_OUT_4), IC1.9 (RF_OUT_1), L15.1, L16.2
- new net: J6.A5 (CC1), R9.1
- new net: C66.1, IC1.8 (2F0)
- new net: C59.2, IC1.3 (RF_IN)
- new net: R19.1, U3.80 (GPIO3)
- new net: C51.1, J6.S1 (SHIELD), R11.1
- new net: IC1.1 (VCC1), L13.2
- new net: C61.1, L11.2, L14.1
- new net: C63.1, IC1.16 (APC1), R14.2
- new net: J6.A4 (VBUS), J6.A9 (VBUS), J6.B4 (VBUS), J6.B9 (VBUS)
- new net Antenna: J5.2, U5.2 (RF1)
- new net Switch: R17.1, R18.2, U5.7 (CTRL)
- new net Switch_Enable: R19.2, R20.2, U5.8 (ENABLE)
- new net TX: C75.2, U5.5 (RF3)
- new net VAPC: R13.1, R15.1, R16.2
- no-connect marks 28 -> 29
Other:
- moved on the sheet: C21, C22, J2, J5, L6, L7, L8
